Commit message: temp check done

File: simple_pendulum_description/urdf/simple_pendulum_editted.xacro (robot description, xacro)
@@ -1,5 +1,5 @@
 <?xml version="1.0" ?>
 <robot name="simple_pendulum_editted" xmlns:xacro="http://www.ros.org/wiki/xacro">
-  <!-- <xacro:include filename="$(find simple_pendulum_description)/urdf/materials.xacro" /> -->
+  <xacro:include filename="$(find simple_pendulum_description)/urdf/materials.xacro" />
   <!-- <xacro:include filename="$(find simple_pendulum_description)/urdf/simple_pendulum_editted.trans" /> -->
   <!-- <xacro:include filename="$(find simple_pendulum_description)/urdf/simple_pendulum_editted.gazebo" /> -->
@@ -13,5 +13,5 @@
       <origin xyz="0 0 0" rpy="0 0 0"/>
       <geometry>
-        <mesh filename="package://simple_pendulum_description/meshes/editted/base_link.stl" scale="0.001 0.001 0.001"/>
+        <mesh filename="file://$(find simple_pendulum_description)/meshes/editted/base_link.stl" scale="0.001 0.001 0.001"/>
       </geometry>
       <material name="silver"/>
@@ -20,5 +20,5 @@
       <origin xyz="0 0 0" rpy="0 0 0"/>
       <geometry>
-        <mesh filename="package://simple_pendulum_description/meshes/editted/base_link.stl" scale="0.001 0.001 0.001"/>
+        <mesh filename="file://$(find simple_pendulum_description)/meshes/editted/base_link.stl" scale="0.001 0.001 0.001"/>
       </geometry>
     </collision>
@@ -33,5 +33,5 @@
       <origin xyz="-0.017 -0.0 -0.69779" rpy="0 0 0"/>
       <geometry>
-        <mesh filename="package://simple_pendulum_description/meshes/editted/tmotor_ak80_64_1.stl" scale="0.001 0.001 0.001"/>
+        <mesh filename="file://$(find simple_pendulum_description)/meshes/editted/tmotor_ak80_64_1.stl" scale="0.001 0.001 0.001"/>
       </geometry>
       <material name="silver"/>
@@ -40,5 +40,5 @@
       <origin xyz="-0.017 -0.0 -0.69779" rpy="0 0 0"/>
       <geometry>
-        <mesh filename="package://simple_pendulum_description/meshes/editted/tmotor_ak80_64_1.stl" scale="0.001 0.001 0.001"/>
+        <mesh filename="file://$(find simple_pendulum_description)/meshes/editted/tmotor_ak80_64_1.stl" scale="0.001 0.001 0.001"/>
       </geometry>
     </collision>
@@ -53,5 +53,5 @@
       <origin xyz="-0.0677 -0.0 -0.69779" rpy="0 0 0"/>
       <geometry>
-        <mesh filename="package://simple_pendulum_description/meshes/editted/pendulum_1.stl" scale="0.001 0.001 0.001"/>
+        <mesh filename="file://$(find simple_pendulum_description)/meshes/editted/pendulum_1.stl" scale="0.001 0.001 0.001"/>
       </geometry>
       <material name="silver"/>
@@ -60,5 +60,5 @@
       <origin xyz="-0.0677 -0.0 -0.69779" rpy="0 0 0"/>
       <geometry>
-        <mesh filename="package://simple_pendulum_description/meshes/editted/pendulum_1.stl" scale="0.001 0.001 0.001"/>
+        <mesh filename="file://$(find simple_pendulum_description)/meshes/editted/pendulum_1.stl" scale="0.001 0.001 0.001"/>
       </geometry>
     </collision>

File: simple_pendulum_description/urdf/simple_pendulum_original.xacro (robot description, xacro)
@@ -1,5 +1,5 @@
 <?xml version="1.0" ?>
 <robot name="simple_pendulum_original" xmlns:xacro="http://www.ros.org/wiki/xacro">
-<!-- <xacro:include filename="$(find simple_pendulum_description)/urdf/materials.xacro" /> -->
+<xacro:include filename="$(find simple_pendulum_description)/urdf/materials.xacro" />
 <!-- <xacro:include filename="$(find simple_pendulum_description)/urdf/simple_pendulum_original.trans" /> -->
 <!-- <xacro:include filename="$(find simple_pendulum_description)/urdf/simple_pendulum_original.gazebo" /> -->
@@ -13,5 +13,5 @@
       <origin xyz="0 0 0" rpy="0 0 0"/>
       <geometry>
-        <mesh filename="package://simple_pendulum_description/meshes/original/base_link.stl" scale="0.001 0.001 0.001"/>
+        <mesh filename="file://$(find simple_pendulum_description)/meshes/original/base_link.stl" scale="0.001 0.001 0.001"/>
       </geometry>
       <material name="silver"/>
@@ -20,5 +20,5 @@
       <origin xyz="0 0 0" rpy="0 0 0"/>
       <geometry>
-        <mesh filename="package://simple_pendulum_description/meshes/original/base_link.stl" scale="0.001 0.001 0.001"/>
+        <mesh filename="file://$(find simple_pendulum_description)/meshes/original/base_link.stl" scale="0.001 0.001 0.001"/>
       </geometry>
     </collision>
@@ -33,5 +33,5 @@
       <origin xyz="0.0 -0.0 -0.037" rpy="0 0 0"/>
       <geometry>
-        <mesh filename="package://simple_pendulum_description/meshes/original/t_motor_ak80_64_body_1.stl" scale="0.001 0.001 0.001"/>
+        <mesh filename="file://$(find simple_pendulum_description)/meshes/original/t_motor_ak80_64_body_1.stl" scale="0.001 0.001 0.001"/>
       </geometry>
       <material name="silver"/>
@@ -40,5 +40,5 @@
       <origin xyz="0.0 -0.0 -0.037" rpy="0 0 0"/>
       <geometry>
-        <mesh filename="package://simple_pendulum_description/meshes/original/t_motor_ak80_64_body_1.stl" scale="0.001 0.001 0.001"/>
+        <mesh filename="file://$(find simple_pendulum_description)/meshes/original/t_motor_ak80_64_body_1.stl" scale="0.001 0.001 0.001"/>
       </geometry>
     </collision>
@@ -53,5 +53,5 @@
       <origin xyz="0.0 0.0 -0.0877" rpy="0 0 0"/>
       <geometry>
-        <mesh filename="package://simple_pendulum_description/meshes/original/pendulum_1.stl" scale="0.001 0.001 0.001"/>
+        <mesh filename="file://$(find simple_pendulum_description)/meshes/original/pendulum_1.stl" scale="0.001 0.001 0.001"/>
       </geometry>
       <material name="silver"/>
@@ -60,5 +60,5 @@
       <origin xyz="0.0 0.0 -0.0877" rpy="0 0 0"/>
       <geometry>
-        <mesh filename="package://simple_pendulum_description/meshes/original/pendulum_1.stl" scale="0.001 0.001 0.001"/>
+        <mesh filename="file://$(find simple_pendulum_description)/meshes/original/pendulum_1.stl" scale="0.001 0.001 0.001"/>
       </geometry>
     </collision>
