Commit message: basic ctrl example for isaac sim added

File: simple_pendulum_description/urdf/simple_pendulum_editted.urdf (robot description, URDF)
Before this commit: robot simple_pendulum_editted, 3 links, 2 joints
Links:
- link base_link: geometry collision mesh filename=package://simple_pendulum_description/meshes/editted/base_l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 scale=0.001 0.001 0.001; visual mesh filename=package://simple_pendulum_description/meshes/editted/base_l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 scale=0.001 0.001 0.001
- link pendulum_1: geometry collision mesh filename=package://simple_pendulum_description/meshes/editted/pendul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 scale=0.001 0.001 0.001; visual mesh filename=package://simple_pendulum_description/meshes/editted/pendul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 scale=0.001 0.001 0.001
- link tmotor_ak80_64_1: geometry collision mesh filename=package://simple_pendulum_description/meshes/editted/tmotor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 scale=0.001 0.001 0.001; visual mesh filename=package://simple_pendulum_description/meshes/editted/tmotor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 scale=0.001 0.001 0.001
