Commit message: urdf first done

File: Fusion2URDF_description/urdf/Fusion2URDF.xacro (robot description, xacro)
@@ -11,5 +11,5 @@
   </inertial>
   <visual>
-    <origin xyz="0.15 0.1 0" rpy="0 0 0"/>
+    <origin xyz="0 0 0" rpy="0 0 0"/>
     <geometry>
       <mesh filename="file://$(find bj_actuator_rviz)/meshes/base_link.stl" scale="0.001 0.001 0.001"/>
@@ -18,5 +18,5 @@
   </visual>
   <collision>
-    <origin xyz="0.15 0.1 0" rpy="0 0 0"/>
+    <origin xyz="0 0 0" rpy="0 0 0"/>
     <geometry>
       <mesh filename="file://$(find bj_actuator_rviz)/meshes/base_link.stl" scale="0.001 0.001 0.001"/>
@@ -31,5 +31,5 @@
   </inertial>
   <visual>
-    <origin xyz="0.15 0.148 -0.02" rpy="0 0 0"/>
+    <origin xyz="-0.0 0.048 -0.02" rpy="0 0 0"/>
     <geometry>
       <mesh filename="file://$(find bj_actuator_rviz)/meshes/motor_mount_1.stl" scale="0.001 0.001 0.001"/>
@@ -38,5 +38,5 @@
   </visual>
   <collision>
-    <origin xyz="0.15 0.148 -0.02" rpy="0 0 0"/>
+    <origin xyz="-0.0 0.048 -0.02" rpy="0 0 0"/>
     <geometry>
       <mesh filename="file://$(find bj_actuator_rviz)/meshes/motor_mount_1.stl" scale="0.001 0.001 0.001"/>
@@ -51,5 +51,5 @@
   </inertial>
   <visual>
-    <origin xyz="0.184875 0.23427 -0.11255" rpy="0 0 0"/>
+    <origin xyz="0.034875 0.13427 -0.11255" rpy="0 0 0"/>
     <geometry>
       <mesh filename="file://$(find bj_actuator_rviz)/meshes/front_case_1.stl" scale="0.001 0.001 0.001"/>
@@ -58,5 +58,5 @@
   </visual>
   <collision>
-    <origin xyz="0.184875 0.23427 -0.11255" rpy="0 0 0"/>
+    <origin xyz="0.034875 0.13427 -0.11255" rpy="0 0 0"/>
     <geometry>
       <mesh filename="file://$(find bj_actuator_rviz)/meshes/front_case_1.stl" scale="0.001 0.001 0.001"/>
@@ -71,5 +71,5 @@
   </inertial>
   <visual>
-    <origin xyz="0.184875 0.21 -0.11255" rpy="0 0 0"/>
+    <origin xyz="0.034875 0.11 -0.11255" rpy="0 0 0"/>
     <geometry>
       <mesh filename="file://$(find bj_actuator_rviz)/meshes/rear_case_241023_1.stl" scale="0.001 0.001 0.001"/>
@@ -78,5 +78,5 @@
   </visual>
   <collision>
-    <origin xyz="0.184875 0.21 -0.11255" rpy="0 0 0"/>
+    <origin xyz="0.034875 0.11 -0.11255" rpy="0 0 0"/>
     <geometry>
       <mesh filename="file://$(find bj_actuator_rviz)/meshes/rear_case_241023_1.stl" scale="0.001 0.001 0.001"/>
@@ -91,5 +91,5 @@
   </inertial>
   <visual>
-    <origin xyz="0.184875 0.27717 0.07745" rpy="0 0 0"/>
+    <origin xyz="0.034875 0.17717 0.07745" rpy="0 0 0"/>
     <geometry>
       <mesh filename="file://$(find bj_actuator_rviz)/meshes/mass_plate_1.stl" scale="0.001 0.001 0.001"/>
@@ -98,5 +98,5 @@
   </visual>
   <collision>
-    <origin xyz="0.184875 0.27717 0.07745" rpy="0 0 0"/>
+    <origin xyz="0.034875 0.17717 0.07745" rpy="0 0 0"/>
     <geometry>
       <mesh filename="file://$(find bj_actuator_rviz)/meshes/mass_plate_1.stl" scale="0.001 0.001 0.001"/>
@@ -111,5 +111,5 @@
   </inertial>
   <visual>
-    <origin xyz="0.184875 0.26687 -0.11255" rpy="0 0 0"/>
+    <origin xyz="0.034875 0.16687 -0.11255" rpy="0 0 0"/>
     <geometry>
       <mesh filename="file://$(find bj_actuator_rviz)/meshes/bearing_1.stl" scale="0.001 0.001 0.001"/>
@@ -118,5 +118,5 @@
   </visual>
   <collision>
-    <origin xyz="0.184875 0.26687 -0.11255" rpy="0 0 0"/>
+    <origin xyz="0.034875 0.16687 -0.11255" rpy="0 0 0"/>
     <geometry>
       <mesh filename="file://$(find bj_actuator_rviz)/meshes/bearing_1.stl" scale="0.001 0.001 0.001"/>
@@ -131,5 +131,5 @@
   </inertial>
   <visual>
-    <origin xyz="0.184875 0.26717 -0.11255" rpy="0 0 0"/>
+    <origin xyz="0.034875 0.16717 -0.11255" rpy="0 0 0"/>
     <geometry>
       <mesh filename="file://$(find bj_actuator_rviz)/meshes/test_bar_1.stl" scale="0.001 0.001 0.001"/>
@@ -138,5 +138,5 @@
   </visual>
   <collision>
-    <origin xyz="0.184875 0.26717 -0.11255" rpy="0 0 0"/>
+    <origin xyz="0.034875 0.16717 -0.11255" rpy="0 0 0"/>
     <geometry>
       <mesh filename="file://$(find bj_actuator_rviz)/meshes/test_bar_1.stl" scale="0.001 0.001 0.001"/>
@@ -149,4 +149,9 @@
   <child link="motor_mount_1"/>
 </joint>
+<joint name="case_joint" type="fixed">
+  <origin xyz="0.0 -0.02427 0.0" rpy="0 0 0"/>
+  <parent link="rear_case_241023_1"/>
+  <child link="front_case_1"/>
+</joint>
 <joint name="mount_joint" type="fixed">
   <origin xyz="-0.034875 -0.062 0.09255" rpy="0 0 0"/>
@@ -154,8 +159,8 @@
   <child link="rear_case_241023_1"/>
 </joint>
-<joint name="case_joint" type="fixed">
-  <origin xyz="0.0 -0.02427 0.0" rpy="0 0 0"/>
-  <parent link="rear_case_241023_1"/>
-  <child link="front_case_1"/>
+<joint name="mass_joint" type="fixed">
+  <origin xyz="0.0 -0.01 -0.19" rpy="0 0 0"/>
+  <parent link="test_bar_1"/>
+  <child link="mass_plate_1"/>
 </joint>
 <joint name="gear_joint" type="fixed">
@@ -164,14 +169,8 @@
   <child link="bearing_1"/>
 </joint>
-<joint name="continuous_joint" type="continuous">
+<joint name="continuous_joint" type="fixed">
   <origin xyz="0.0 -0.0003 0.0" rpy="0 0 0"/>
   <parent link="bearing_1"/>
   <child link="test_bar_1"/>
-  <axis xyz="0.0 1.0 0.0"/>
-</joint>
-<joint name="mass_joint" type="fixed">
-  <origin xyz="0.0 -0.01 -0.19" rpy="0 0 0"/>
-  <parent link="test_bar_1"/>
-  <child link="mass_plate_1"/>
 </joint>
 </robot>
